Commit message: proper formatting

File: ws/wheel_bot/urdf/four_wheel_bot.xacro (robot description, xacro)
@@ -1,7 +1,4 @@
 <?xml version="1.0" ?>
 <robot name="four_wheel_bot" xmlns:xacro="http://www.ros.org/wiki/xacro">
-<xacro:include filename="$(find four_wheel_bot_description)/urdf/materials.xacro" />
-<xacro:include filename="$(find four_wheel_bot_description)/urdf/four_wheel_bot.trans" />
-<xacro:include filename="$(find four_wheel_bot_description)/urdf/ros2_control.xacro" />
 <link name="base_link">
   <inertial>
@@ -13,12 +10,11 @@
     <origin xyz="0 0 0" rpy="0 0 0"/>
     <geometry>
-      <mesh filename="file://$(find four_wheel_bot_description)/meshes/base_link.stl" scale="0.001 0.001 0.001"/>
+      <mesh filename="meshes/base_link.stl" scale="0.001 0.001 0.001"/>
     </geometry>
-    <material name="silver"/>
   </visual>
   <collision>
     <origin xyz="0 0 0" rpy="0 0 0"/>
     <geometry>
-      <mesh filename="file://$(find four_wheel_bot_description)/meshes/base_link.stl" scale="0.001 0.001 0.001"/>
+      <mesh filename="meshes/base_link.stl" scale="0.001 0.001 0.001"/>
     </geometry>
   </collision>
@@ -33,12 +29,11 @@
     <origin xyz="-0.04 -0.035 -0.015" rpy="0 0 0"/>
     <geometry>
-      <mesh filename="file://$(find four_wheel_bot_description)/meshes/left_front_wheel_1.stl" scale="0.001 0.001 0.001"/>
+      <mesh filename="meshes/left_front_wheel_1.stl" scale="0.001 0.001 0.001"/>
     </geometry>
-    <material name="silver"/>
   </visual>
   <collision>
     <origin xyz="-0.04 -0.035 -0.015" rpy="0 0 0"/>
     <geometry>
-      <mesh filename="file://$(find four_wheel_bot_description)/meshes/left_front_wheel_1.stl" scale="0.001 0.001 0.001"/>
+      <mesh filename="meshes/left_front_wheel_1.stl" scale="0.001 0.001 0.001"/>
     </geometry>
   </collision>
@@ -53,12 +48,11 @@
     <origin xyz="0.04 -0.035 -0.015" rpy="0 0 0"/>
     <geometry>
-      <mesh filename="file://$(find four_wheel_bot_description)/meshes/left_back_wheel_1.stl" scale="0.001 0.001 0.001"/>
+      <mesh filename="meshes/left_back_wheel_1.stl" scale="0.001 0.001 0.001"/>
     </geometry>
-    <material name="silver"/>
   </visual>
   <collision>
     <origin xyz="0.04 -0.035 -0.015" rpy="0 0 0"/>
     <geometry>
-      <mesh filename="file://$(find four_wheel_bot_description)/meshes/left_back_wheel_1.stl" scale="0.001 0.001 0.001"/>
+      <mesh filename="meshes/left_back_wheel_1.stl" scale="0.001 0.001 0.001"/>
     </geometry>
   </collision>
@@ -73,12 +67,11 @@
     <origin xyz="-0.04 0.035 -0.015" rpy="0 0 0"/>
     <geometry>
-      <mesh filename="file://$(find four_wheel_bot_description)/meshes/right_front_wheel_1.stl" scale="0.001 0.001 0.001"/>
+      <mesh filename="meshes/right_front_wheel_1.stl" scale="0.001 0.001 0.001"/>
     </geometry>
-    <material name="silver"/>
   </visual>
   <collision>
     <origin xyz="-0.04 0.035 -0.015" rpy="0 0 0"/>
     <geometry>
-      <mesh filename="file://$(find four_wheel_bot_description)/meshes/right_front_wheel_1.stl" scale="0.001 0.001 0.001"/>
+      <mesh filename="meshes/right_front_wheel_1.stl" scale="0.001 0.001 0.001"/>
     </geometry>
   </collision>
@@ -93,12 +86,11 @@
     <origin xyz="0.04 0.035 -0.015" rpy="0 0 0"/>
     <geometry>
-      <mesh filename="file://$(find four_wheel_bot_description)/meshes/right_back_wheel_1.stl" scale="0.001 0.001 0.001"/>
+      <mesh filename="meshes/right_back_wheel_1.stl" scale="0.001 0.001 0.001"/>
     </geometry>
-    <material name="silver"/>
   </visual>
   <collision>
     <origin xyz="0.04 0.035 -0.015" rpy="0 0 0"/>
     <geometry>
-      <mesh filename="file://$(find four_wheel_bot_description)/meshes/right_back_wheel_1.stl" scale="0.001 0.001 0.001"/>
+      <mesh filename="meshes/right_back_wheel_1.stl" scale="0.001 0.001 0.001"/>
     </geometry>
   </collision>
@@ -113,12 +105,11 @@
     <origin xyz="-0.051 -0.0 -0.025" rpy="0 0 0"/>
     <geometry>
-      <mesh filename="file://$(find four_wheel_bot_description)/meshes/camera_sensor_1.stl" scale="0.001 0.001 0.001"/>
+      <mesh filename="meshes/camera_sensor_1.stl" scale="0.001 0.001 0.001"/>
     </geometry>
-    <material name="silver"/>
   </visual>
   <collision>
     <origin xyz="-0.051 -0.0 -0.025" rpy="0 0 0"/>
     <geometry>
-      <mesh filename="file://$(find four_wheel_bot_description)/meshes/camera_sensor_1.stl" scale="0.001 0.001 0.001"/>
+      <mesh filename="meshes/camera_sensor_1.stl" scale="0.001 0.001 0.001"/>
     </geometry>
   </collision>
@@ -133,12 +124,11 @@
     <origin xyz="-0.0 -0.0 -0.055" rpy="0 0 0"/>
     <geometry>
-      <mesh filename="file://$(find four_wheel_bot_description)/meshes/lidar_sensor_1.stl" scale="0.001 0.001 0.001"/>
+      <mesh filename="meshes/lidar_sensor_1.stl" scale="0.001 0.001 0.001"/>
     </geometry>
-    <material name="silver"/>
   </visual>
   <collision>
     <origin xyz="-0.0 -0.0 -0.055" rpy="0 0 0"/>
     <geometry>
-      <mesh filename="file://$(find four_wheel_bot_description)/meshes/lidar_sensor_1.stl" scale="0.001 0.001 0.001"/>
+      <mesh filename="meshes/lidar_sensor_1.stl" scale="0.001 0.001 0.001"/>
     </geometry>
   </collision>
